Commit message: New Joint in inter_5

File: ros2_ws/iteration_5/urdf/moveo.ros2_control.xacro (robot description, xacro)
@@ -33,4 +33,16 @@
 				<state_interface name="velocity"/>
 			</joint>
+			<joint name="Joint_3">
+				<param name="id">3</param>
+				<param name="pin_pulse">44</param>
+				<param name="pin_dir">42</param>
+				<param name="direction">1</param>
+				<param name="steps_per_revolution">256</param>
+				<param name="encoder_i2c_adress">0x48</param>
+				<param name="initial_position_offset">0</param>
+				<command_interface name="velocity"/>
+				<state_interface name="position"/>
+				<state_interface name="velocity"/>
+			</joint>
 		</ros2_control>
 </robot>

File: ros2_ws/iteration_5/urdf/moveo.urdf (robot description, URDF)
Before this commit: robot moveo, 4 links, 3 joints
Links:
- added link Link_3, mass 1.2; collision mesh filename=package://iteration_3/meshes/Link_3.stl; visual mesh filename=package://iteration_3/meshes/Link_3.stl
Joints:
- added joint Joint_3: type revolute, parent Link_2, child Link_3, origin xyz=0 0 0.221 rpy=0 0 0, axis -1 0 0, limit lower=-1.963 upper=1.963 effort=5.0 velocity=1.0
